Commit message: ir sensor added , maybe add 3 more ir sensors

File: fb_description/urdf/fb.xacro (robot description, xacro)
@@ -51,4 +51,23 @@
     </inertial>
   </link>
+  <link name="base_ir_front">
+    <collision>
+      <origin xyz="0 0 0" rpy="0 0 0"/>
+      <geometry>
+        <box size="0.01 0.01 0.01"/>
+      </geometry>
+    </collision>
+    <visual>
+      <origin xyz="0 0 0" rpy="0 0 0"/>
+      <geometry>
+        <box size="0.01 0.01 0.01"/>
+      </geometry>
+    </visual>
+    <inertial>
+      <mass value="1e-5" />
+      <origin xyz="0 0 0" rpy="0 0 0"/>
+      <inertia ixx="1e-6" ixy="0" ixz="0" iyy="1e-6" iyz="0"      izz="1e-6" />
+    </inertial>
+</link>
   <link name="right_wheel">
     <!--origin xyz="0.1 -0.13 0.1" rpy="0 1.5707 1.5707"/-->
@@ -123,5 +142,11 @@
     </inertial>
   </link>
-  <joint type="continuous" name="left_wheel_hinge">
+ <joint name="ir_front_joint" type="fixed">
+    <axis xyz="0 1 0" />
+    <origin rpy="0 0 0" xyz="0.2 0.02 0.020" />
+    <parent link="chassis"/>
+    <child link="base_ir_front"/>
+</joint>
+ <joint type="continuous" name="left_wheel_hinge">
     <origin xyz="0.2 0.15 0" rpy="0 0 0"/>
     <child link="left_wheel"/>

Commit message: added imu in gazebo as well , angulat v is not correct

File: fb_description/urdf/fb.xacro (robot description, xacro)
@@ -70,4 +70,23 @@
     </inertial>
 </link>
+  <link name="imu_link">
+    <collision>
+      <origin xyz="0 0 0" rpy="0 0 0"/>
+      <geometry>
+        <box size="0.01 0.01 0.01"/>
+      </geometry>
+    </collision>
+    <visual>
+      <origin xyz="0 0 0" rpy="0 0 0"/>
+      <geometry>
+        <box size="0.01 0.01 0.01"/>
+      </geometry>
+    </visual>
+    <inertial>
+      <mass value="1e-5" />
+      <origin xyz="0 0 0" rpy="0 0 0"/>
+      <inertia ixx="1e-6" ixy="0" ixz="0" iyy="1e-6" iyz="0"      izz="1e-6" />
+    </inertial>
+</link>
   <link name="right_wheel">
     <!--origin xyz="0.1 -0.13 0.1" rpy="0 1.5707 1.5707"/-->
@@ -147,4 +166,10 @@
     <parent link="chassis"/>
     <child link="base_ir_front"/>
+</joint>
+<joint name="imu_joint" type="fixed">
+    <axis xyz="0 1 0" />
+    <origin rpy="0 1.57 0" xyz="0.1 0.02 0.05" />
+    <parent link="chassis"/>
+    <child link="imu_link"/>
 </joint>
  <joint type="continuous" name="left_wheel_hinge">

Commit message: added rover branch , realsense camera , bug:pointcloud publishing perpendicular

File: fb_description/urdf/fb.xacro (robot description, xacro)
@@ -51,5 +51,5 @@
     </inertial>
   </link>
-  <link name="base_ir_front">
+  <link name="rgbd">
     <collision>
       <origin xyz="0 0 0" rpy="0 0 0"/>
@@ -161,9 +161,9 @@
     </inertial>
   </link>
- <joint name="ir_front_joint" type="fixed">
-    <axis xyz="0 1 0" />
+ <joint name="camera_joint" type="fixed">
+    <axis xyz="0 0 0" />
     <origin rpy="0 0 0" xyz="0.2 0.02 0.020" />
     <parent link="chassis"/>
-    <child link="base_ir_front"/>
+    <child link="rgbd"/>
 </joint>
 <joint name="imu_joint" type="fixed">

Commit message: everything is working fine , added rviz launch file

File: fb_description/urdf/fb.xacro (robot description, xacro)
@@ -4,4 +4,8 @@
   <xacro:include filename="$(find fb_description)/urdf/materials.xacro" />
   <!--xacro:include filename="$(find mybot_description)/urdf/macros.xacro" /-->
+ <xacro:property name="r200_cam_rgb_px" value="0.05"/>
+  <xacro:property name="r200_cam_rgb_py" value="0.018"/>
+  <xacro:property name="r200_cam_rgb_pz" value="0.013"/>
+  <xacro:property name="r200_cam_depth_offset" value="0.01"/>
   <link name='chassis'>
     <pose>0 0 0.1 0 0 0</pose>
@@ -51,6 +55,57 @@
     </inertial>
   </link>
-  <link name="rgbd">
+   <joint name="camera_joint" type="fixed">
+    <origin xyz="0.22 -0.07 0.04" rpy="0 0 0"/>
+    <parent link="chassis"/>
+    <child link="camera_link"/>
+  </joint>
+  <link name="camera_link">
+    <visual>
+     <origin xyz="0 0 0" rpy="1.57 0 1.57"/>
+      <geometry>
+       <mesh filename="/home/manan/catkin_ws/src/final_bot/fb_description/urdf/r200.dae"/>
+      </geometry>
+    </visual>
     <collision>
+      <origin xyz="0.003 0.065 0.007" rpy="0 0 0"/>
+      <geometry>
+        <box size="0.012 0.132 0.020"/>
+      </geometry>
+    </collision>
+    <!-- This inertial field needs doesn't contain reliable data!! -->
+<!--   <inertial>
+      <mass value="0.564" />
+      <origin xyz="0 0 0" />
+      <inertia ixx="0.003881243" ixy="0.0" ixz="0.0"
+               iyy="0.000498940" iyz="0.0"
+               izz="0.003879257" />
+    </inertial>-->
+  </link>
+  <joint name="camera_rgb_joint" type="fixed">
+    <origin xyz="${r200_cam_rgb_px} ${r200_cam_rgb_py} ${r200_cam_rgb_pz}" rpy="0 0 0"/>
+    <parent link="camera_link"/>
+    <child link="camera_rgb_frame"/>
+  </joint>
+  <link name="camera_rgb_frame"/>
+  <joint name="camera_rgb_optical_joint" type="fixed">
+    <origin xyz="0 0 0" rpy="-1.57 0 -1.57"/>
+    <parent link="camera_rgb_frame"/>
+    <child link="camera_rgb_optical_frame"/>
+  </joint>
+  <link name="camera_rgb_optical_frame"/>
+  <joint name="camera_depth_joint" type="fixed">
+    <origin xyz="${r200_cam_rgb_px} ${r200_cam_rgb_py + r200_cam_depth_offset} ${r200_cam_rgb_pz}" rpy="0 0 0"/>
+    <parent link="camera_link"/>
+    <child link="camera_depth_frame"/>
+  </joint>
+  <link name="camera_depth_frame"/>
+  <joint name="camera_depth_optical_joint" type="fixed">
+    <origin xyz="0 0 0" rpy="-1.57 0 -1.57"/>
+    <parent link="camera_depth_frame"/>
+    <child link="camera_depth_optical_frame"/>
+  </joint>
+  <link name="camera_depth_optical_frame"/>
+  <!-- <link name="rgbd">
+    <collision>
       <origin xyz="0 0 0" rpy="0 0 0"/>
       <geometry>
@@ -59,5 +114,5 @@
     </collision>
     <visual>
-      <origin xyz="0 0 0" rpy="0 0 0"/>
+      <origin xyz="0 0 0" rpy="-1.5708 0 -1.5708"/>
       <geometry>
         <box size="0.01 0.01 0.01"/>
@@ -69,5 +124,5 @@
       <inertia ixx="1e-6" ixy="0" ixz="0" iyy="1e-6" iyz="0"      izz="1e-6" />
     </inertial>
-</link>
+</link> -->
   <link name="imu_link">
     <collision>
@@ -161,4 +216,5 @@
     </inertial>
   </link>
+ <!--
  <joint name="camera_joint" type="fixed">
     <axis xyz="0 0 0" />
@@ -167,7 +223,8 @@
     <child link="rgbd"/>
 </joint>
+-->
 <joint name="imu_joint" type="fixed">
-    <axis xyz="0 1 0" />
-    <origin rpy="0 1.57 0" xyz="0.1 0.02 0.05" />
+    <axis xyz="0 0 0" />
+    <origin rpy="0 1.57 0" xyz="0.1 0 0.05" />
     <parent link="chassis"/>
     <child link="imu_link"/>

Commit message: updated readme and other things

File: fb_description/urdf/fb.xacro (robot description, xacro)
@@ -70,4 +70,61 @@
     </inertial>
 </link>
+  <link name="base_ir_back">
+    <collision>
+      <origin xyz="0 0 0" rpy="0 0 0"/>
+      <geometry>
+        <box size="0.01 0.01 0.01"/>
+      </geometry>
+    </collision>
+    <visual>
+      <origin xyz="0 0 0" rpy="0 0 0"/>
+      <geometry>
+        <box size="0.01 0.01 0.01"/>
+      </geometry>
+    </visual>
+    <inertial>
+      <mass value="1e-5" />
+      <origin xyz="0 0 0" rpy="0 0 0"/>
+      <inertia ixx="1e-6" ixy="0" ixz="0" iyy="1e-6" iyz="0"      izz="1e-6" />
+    </inertial>
+</link>
+  <link name="base_ir_side1">
+    <collision>
+      <origin xyz="0 0 0" rpy="0 0 0"/>
+      <geometry>
+        <box size="0.01 0.01 0.01"/>
+      </geometry>
+    </collision>
+    <visual>
+      <origin xyz="0 0 0" rpy="0 0 0"/>
+      <geometry>
+        <box size="0.01 0.01 0.01"/>
+      </geometry>
+    </visual>
+    <inertial>
+      <mass value="1e-5" />
+      <origin xyz="0 0 0" rpy="0 0 0"/>
+      <inertia ixx="1e-6" ixy="0" ixz="0" iyy="1e-6" iyz="0"      izz="1e-6" />
+    </inertial>
+</link>
+  <link name="base_ir_side2">
+    <collision>
+      <origin xyz="0 0 0" rpy="0 0 0"/>
+      <geometry>
+        <box size="0.01 0.01 0.01"/>
+      </geometry>
+    </collision>
+    <visual>
+      <origin xyz="0 0 0" rpy="0 0 0"/>
+      <geometry>
+        <box size="0.01 0.01 0.01"/>
+      </geometry>
+    </visual>
+    <inertial>
+      <mass value="1e-5" />
+      <origin xyz="0 0 0" rpy="0 0 0"/>
+      <inertia ixx="1e-6" ixy="0" ixz="0" iyy="1e-6" iyz="0"      izz="1e-6" />
+    </inertial>
+</link>
   <link name="imu_link">
     <collision>
@@ -166,4 +223,22 @@
     <parent link="chassis"/>
     <child link="base_ir_front"/>
+</joint>
+ <joint name="ir_back_joint" type="fixed">
+    <axis xyz="0 1 0" />
+    <origin rpy="0 0 -3.14" xyz="-0.2 0.02 0.020" />
+    <parent link="chassis"/>
+    <child link="base_ir_back"/>
+</joint>
+ <joint name="ir_side1" type="fixed">
+    <axis xyz="0 1 0" />
+    <origin rpy="0 0 1.57" xyz="0.0 0.1 0.020" />
+    <parent link="chassis"/>
+    <child link="base_ir_side1"/>
+</joint>
+<joint name="ir_side2" type="fixed">
+    <axis xyz="0 1 0" />
+    <origin rpy="0 0 -1.57" xyz="0.0 -0.1 0.020" />
+    <parent link="chassis"/>
+    <child link="base_ir_side2"/>
 </joint>
 <joint name="imu_joint" type="fixed">

Commit message: rviz bugs resolved

File: fb_description/urdf/fb.xacro (robot description, xacro)
@@ -64,5 +64,5 @@
      <origin xyz="0 0 0" rpy="1.57 0 1.57"/>
       <geometry>
-       <mesh filename="/home/manan/catkin_ws/src/final_bot/fb_description/urdf/r200.dae"/>
+       <mesh filename="/home/manan/catkin_ws/src/robot-simulation/fb_description/urdf/r200.dae"/>
       </geometry>
     </visual>

Commit message: simulation

File: fb_description/urdf/fb.xacro (robot description, xacro)
@@ -64,5 +64,5 @@
      <origin xyz="0 0 0" rpy="1.57 0 1.57"/>
       <geometry>
-       <mesh filename="/home/manan/catkin_ws/src/robot-simulation/fb_description/urdf/r200.dae"/>
+       <mesh filename="$(find fb_description)/urdf/r200.dae"/>
       </geometry>
     </visual>
